File: Astable mv.kicad_sch (KiCad schematic)
At the start: 4 parts

Commit message: update
Parts:
- R_Potentiometer_Trim: renamed from RV?; value R_Potentiometer_Trim -> 10k
- gave numbers to parts that had none: 1
Changed lines of the file:
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@@
 		(on_board yes)
 		(dnp no)
-		(fields_autoplaced yes)
-		(property "Reference" "RV?"
-			(at 171.45 93.9799 0)
+		(property "Reference" "R_Potentiometer_Trim"
+			(at 171.196 93.98 0)
 			(effects
 				(font
@@
 			)
 		)
-		(property "Value" "R_Potentiometer_Trim"
-			(at 171.45 96.5199 0)
+		(property "Value" "10k"
+			(at 168.91 96.52 90)
 			(effects
 				(font
@@
 			(project ""
 				(path "/b9aff4a0-d82a-4bce-ac01-704fb6f0f3d4/2d1c429d-f183-4bcd-93b1-5f80de84f69f"
-					(reference "RV?")
+					(reference "R_Potentiometer_Trim")
 					(unit 1)
 				)
@@
 		(dnp no)
 		(fields_autoplaced yes)
-		(property "Reference" "U?"
+		(property "Reference" "U2"
 			(at 149.5141 82.55 0)
 			(effects
@@
 			(project "TENS Device"
 				(path "/b9aff4a0-d82a-4bce-ac01-704fb6f0f3d4/2d1c429d-f183-4bcd-93b1-5f80de84f69f"
-					(reference "U?")
+					(reference "U2")
 					(unit 1)
 				)
