File: Inverter.kicad_sch (KiCad schematic)
At the start: 8 parts

Commit message: preRelease 0.1.0
Changed lines of the file:
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@@
-		)
-	)
-	(global_label "Vin"
-		(shape input)
-		(at 143.51 71.12 90)
-		(fields_autoplaced yes)
-		(effects
-			(font
-				(size 1.27 1.27)
-			)
-			(justify left)
-		)
-		(property "Intersheetrefs" "${INTERSHEET_REFS}"
-			(at 143.51 65.2924 90)
-			(effects
-				(font
-					(size 1.27 1.27)
-				)
-				(justify left)
-				(hide yes)
-			)
 		)
 	)
@@
 		)
 	)
+	(hierarchical_label "Vin"
+		(shape input)
+		(at 143.51 71.12 90)
+		(fields_autoplaced yes)
+		(effects
+			(font
+				(size 1.27 1.27)
+			)
+			(justify left)
+		)
+	)

Commit message: update
Parts:
- gave numbers to parts that had none: 4
Changed lines of the file:
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@@
 		(on_board yes)
 		(dnp no)
-		(fields_autoplaced yes)
-		(property "Reference" "Q?"
-			(at 138.43 111.7599 0)
+		(property "Reference" "Q1"
+			(at 136.652 110.236 0)
 			(effects
 				(font
@@
 			(project "TENS Device"
 				(path "/b9aff4a0-d82a-4bce-ac01-704fb6f0f3d4/bfdd6686-5c44-4050-9e42-e0bc0e78ace7"
-					(reference "Q?")
+					(reference "Q1")
 					(unit 1)
 				)
@@
 		(dnp no)
 		(fields_autoplaced yes)
-		(property "Reference" "Q?"
+		(property "Reference" "Q2"
 			(at 149.86 111.7599 0)
 			(effects
@@
 			(project "TENS Device"
 				(path "/b9aff4a0-d82a-4bce-ac01-704fb6f0f3d4/bfdd6686-5c44-4050-9e42-e0bc0e78ace7"
-					(reference "Q?")
+					(reference "Q2")
 					(unit 1)
 				)
@@
 		(on_board yes)
 		(dnp no)
-		(property "Reference" "R_f?"
+		(property "Reference" "R_f"
 			(at 157.226 78.74 90)
 			(effects
@@
 			(project "TENS Device"
 				(path "/b9aff4a0-d82a-4bce-ac01-704fb6f0f3d4/bfdd6686-5c44-4050-9e42-e0bc0e78ace7"
-					(reference "R_f?")
+					(reference "R_f")
 					(unit 1)
 				)
@@
 		(on_board yes)
 		(dnp no)
-		(property "Reference" "Q?"
-			(at 140.97 80.0099 0)
+		(property "Reference" "Q3"
+			(at 141.224 79.756 0)
 			(effects
 				(font
@@
 			(project "TENS Device"
 				(path "/b9aff4a0-d82a-4bce-ac01-704fb6f0f3d4/bfdd6686-5c44-4050-9e42-e0bc0e78ace7"
-					(reference "Q?")
-					(unit 1)
-				)
+					(reference "Q3")
+					(unit 1)
+				)
