File: untitled.kicad_sch (KiCad schematic)
At the start: 2 parts

Commit message: update
Changed lines of the file:
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@@
 		(on_board yes)
 		(dnp no)
-		(fields_autoplaced yes)
 		(property "Reference" "U3"
-			(at 157.48 95.1201 0)
+			(at 132.08 91.694 0)
 			(effects
 				(font
