File: TENS Device.kicad_sch (KiCad schematic)
At the start: 3 parts, among them SW1 SW_Push

Commit message: update
Parts:
- removed Q?: NPN, symbol Simulation_SPICE:NPN
- removed R_b1: 470, symbol Device:R
Other:
- sheet Astable Multivibrator ports: added RST; removed gnd_reference
